File: RadarInterfaceBoard/RadarFilter-REU2024.kicad_pcb (KiCad board)
At the start: 2 copper layers, 87.4 x 57 mm, 33 parts, among them J1 73099-0, J2 73099-0, J3 73099-0, J4 Conn_01x04_Pin, J5 Conn_01x04_Pin, J6 CONSMA002, J7 CONSMA002, J8 CONSMA002, J9 CONSMA002, U5 ADA4807-2ARM, U6 ADA4807-2ARM

Commit message: fixed op-amp gain
Parts:
- R3, R5, R7, R9: value 10k -> 1k
